File: PACS_1.0/PACS_1.0_power.kicad_sch (KiCad schematic)
At the start: 22 parts, among them Q3 NPN, U2 TPS562201DDCR, U6 S-1011A70-M6T1U4, U7 BSS84PH6327XTSA2

Commit message: Finished Voltage Divider
Parts:
- removed Q3: NPN, symbol Simulation_SPICE:NPN
- added Q2: PN2222A, Package_TO_SOT_THT:TO-92_Inline, symbol Transistor_BJT:PN2222A
- R10: value R -> 10k
- R15: value R -> 5.5k
- R16: value R -> 6.65k
- R17: value R -> 100k
- R18: value R -> 4.7k
Connections:
- net GND: now also Q2.1 (E)
- net at R17.1, R18.2: now also Q2.2 (B)
- net at R10.2, U7.1: now also Q2.3 (C)
Changed lines of the file:
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@@
 			)
 		)
-		(property "Value" "R"
+		(property "Value" "4.7k"
 			(at 156.21 123.19 90)
 			(effects
@@
 	)
 	(symbol
+		(lib_id "Transistor_BJT:PN2222A")
+		(at 179.07 127 0)
+		(unit 1)
+		(exclude_from_sim no)
+		(in_bom yes)
+		(on_board yes)
+		(dnp no)
+		(fields_autoplaced yes)
+		(property "Reference" "Q2"
+			(at 184.15 125.7299 0)
+			(effects
+				(font
+					(size 1.27 1.27)
+				)
+				(justify left)
+			)
+		)
+		(property "Value" "PN2222A"
+			(at 184.15 128.2699 0)
+			(effects
+				(font
+					(size 1.27 1.27)
+				)
+				(justify left)
+			)
+		)
+		(property "Footprint" "Package_TO_SOT_THT:TO-92_Inline"
+			(at 184.15 128.905 0)
+			(effects
+				(font
+					(size 1.27 1.27)
+					(italic yes)
+				)
+				(justify left)
+				(hide yes)
+			)
+		)
+		(property "Datasheet" "https://www.onsemi.com/pub/Collateral/PN2222-D.PDF"
+			(at 179.07 127 0)
+			(effects
+				(font
+					(size 1.27 1.27)
+				)
+				(justify left)
+				(hide yes)
+			)
+		)
+		(property "Description" "1A Ic, 40V Vce, NPN Transistor, General Purpose Transistor, TO-92"
+			(at 179.07 127 0)
+			(effects
+				(font
+					(size 1.27 1.27)
+				)
+				(hide yes)
+			)
+		)
+		(pin "2"
+		)
+		(pin "1"
+		)
+		(pin "3"
+		)
+		(instances
+			(project ""
+				(path "/6996cbc8-fffb-40fd-8350-2bb7d19e6e7a/dd51c51a-fa64-4ebf-8f16-6468af1aee8c"
+					(reference "Q2")
+					(unit 1)
+				)
+			)
+		)
+	)
+	(symbol
 		(lib_id "Device:Battery")
 		(at 33.02 57.15 0)
@@
 			)
 		)
-		(property "Value" "R"
+		(property "Value" "100k"
 			(at 168.91 135.8899 0)
 			(effects
@@
 			)
 		)
-		(property "Value" "R"
+		(property "Value" "6.65k"
 			(at 208.28 146.0499 0)
 			(effects
@@
 	)
 	(symbol
-		(lib_id "Simulation_SPICE:NPN")
-		(at 179.07 127 0)
-		(unit 1)
-		(exclude_from_sim no)
-		(in_bom yes)
-		(on_board yes)
-		(dnp no)
-		(fields_autoplaced yes)
-		(property "Reference" "Q3"
-			(at 184.15 125.7299 0)
-			(effects
-				(font
-					(size 1.27 1.27)
-				)
-				(justify left)
-			)
-		)
-		(property "Value" "NPN"
-			(at 184.15 128.2699 0)
-			(effects
-				(font
-					(size 1.27 1.27)
-				)
-				(justify left)
-			)
-		)
-		(property "Footprint" ""
-			(at 242.57 127 0)
-			(effects
-				(font
-					(size 1.27 1.27)
-				)
-				(hide yes)
-			)
-		)
-		(property "Datasheet" "https://ngspice.sourceforge.io/docs/ngspice-html-manual/manual.xhtml#cha_BJTs"
-			(at 242.57 127 0)
-			(effects
-				(font
-					(size 1.27 1.27)
-				)
-				(hide yes)
-			)
-		)
-		(property "Description" "Bipolar transistor symbol for simulation only, substrate tied to the emitter"
-			(at 179.07 127 0)
-			(effects
-				(font
-					(size 1.27 1.27)
-				)
-				(hide yes)
-			)
-		)
-		(property "Sim.Device" "NPN"
-			(at 179.07 127 0)
-			(effects
-				(font
-					(size 1.27 1.27)
-				)
-				(hide yes)
-			)
-		)
-		(property "Sim.Type" "GUMMELPOON"
-			(at 179.07 127 0)
-			(effects
-				(font
-					(size 1.27 1.27)
-				)
-				(hide yes)
-			)
-		)
-		(property "Sim.Pins" "1=C 2=B 3=E"
-			(at 179.07 127 0)
-			(effects
-				(font
-					(size 1.27 1.27)
-				)
-				(hide yes)
-			)
-		)
-		(pin "3"
-		)
-		(pin "2"
-		)
-		(pin "1"
-		)
-		(instances
-			(project ""
-				(path "/6996cbc8-fffb-40fd-8350-2bb7d19e6e7a/dd51c51a-fa64-4ebf-8f16-6468af1aee8c"
-					(reference "Q3")
-					(unit 1)
-				)
-			)
-		)
-	)
-	(symbol
 		(lib_id "Device:R")
 		(at 172.72 71.12 0)
@@
 			)
 		)
-		(property "Value" "R"
+		(property "Value" "5.5k"
 			(at 208.28 130.8099 0)
 			(effects
@@
 			)
 		)
-		(property "Value" "R"
+		(property "Value" "10k"
 			(at 184.15 109.2199 0)
 			(effects

Commit message: COMPLETE PACS v1.0
Parts:
- removed U6: S-1011A70-M6T1U4, SOT236-A-PKG_MP006-A-P-SD-2.1_ABL, symbol S-1011A70-M6T1U4:S-1011A70-M6T1U4
- added U8: S-80855CNMC-B9GT2U, Package_TO_SOT_SMD:SOT-23-5, symbol S-80855CNMC-B9GT2U:S-80855CNMC-B9GT2U
- R16: value 6.65k -> 5.76k
Connections:
- net GND: now also U8.3 (VSS), U8.4 (NC), U8.5 (NC)
- net at R12.2, R3.1: now also U8.1 (OUT)
- net at C7.1, C8.1, C9.1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: now also U8.2 (VDD)
- no-connect marks 2 -> 0

Commit message: Changed reference for Components
C8 to C2 (AS EXAMPLE)
Parts:
- renumbered C6 to C10, C7 to C5, C8 to C6, C9 to C7, C4 to C8, C5 to C9, Q2 to Q1, R1 to R10, R15 to R11, R16 to R12, R12 to R4, R18 to R5, R3 to R6, R17 to R7, R2 to R8, R10 to R9, U8 to U2, U7 to U3, U2 to U4
Changed lines of the file:
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@@
 		(on_board yes)
 		(dnp no)
-		(property "Reference" "R3"
+		(property "Reference" "R6"
 			(at 166.37 55.88 90)
 			(effects
@@
 			(project "PACS_1.0"
 				(path "/6996cbc8-fffb-40fd-8350-2bb7d19e6e7a/dd51c51a-fa64-4ebf-8f16-6468af1aee8c"
-					(reference "R3")
+					(reference "R6")
 					(unit 1)
 				)
@@
 		(dnp no)
 		(fields_autoplaced yes)
-		(property "Reference" "C8"
+		(property "Reference" "C6"
 			(at 172.72 39.3701 0)
 			(effects
@@
 			(project "PACS_1.0"
 				(path "/6996cbc8-fffb-40fd-8350-2bb7d19e6e7a/dd51c51a-fa64-4ebf-8f16-6468af1aee8c"
-					(reference "C8")
+					(reference "C6")
 					(unit 1)
 				)
@@
 		(dnp no)
 		(fields_autoplaced yes)
-		(property "Reference" "#PWR035"
+		(property "Reference" "#PWR015"
 			(at 181.61 154.94 0)
 			(effects
@@
 			(project ""
 				(path "/6996cbc8-fffb-40fd-8350-2bb7d19e6e7a/dd51c51a-fa64-4ebf-8f16-6468af1aee8c"
-					(reference "#PWR035")
+					(reference "#PWR015")
 					(unit 1)
 				)
@@
 		(on_board yes)
 		(dnp no)
-		(property "Reference" "#PWR06"
+		(property "Reference" "#PWR018"
 			(at 229.87 76.2 0)
 			(effects
@@
 			(project ""
 				(path "/6996cbc8-fffb-40fd-8350-2bb7d19e6e7a/dd51c51a-fa64-4ebf-8f16-6468af1aee8c"
-					(reference "#PWR06")
+					(reference "#PWR018")
 					(unit 1)
 				)
@@
 		(dnp no)
 		(fields_autoplaced yes)
-		(property "Reference" "R18"
+		(property "Reference" "R5"
 			(at 156.21 120.65 90)
 			(effects
@@
 			(project "PACS_1.0"
 				(path "/6996cbc8-fffb-40fd-8350-2bb7d19e6e7a/dd51c51a-fa64-4ebf-8f16-6468af1aee8c"
-					(reference "R18")
+					(reference "R5")
 					(unit 1)
 				)
@@
 		(on_board yes)
 		(dnp no)
-		(property "Reference" "R12"
+		(property "Reference" "R4"
 			(at 101.6 101.6 90)
 			(effects
@@
 			(project "PACS_1.0"
 				(path "/6996cbc8-fffb-40fd-8350-2bb7d19e6e7a/dd51c51a-fa64-4ebf-8f16-6468af1aee8c"
-					(reference "R12")
+					(reference "R4")
 					(unit 1)
 				)
@@
 		(on_board yes)
 		(dnp no)
-		(property "Reference" "C4"
+		(property "Reference" "C8"
 			(at 212.09 81.788 90)
 			(effects
@@
 			(project ""
 				(path "/6996cbc8-fffb-40fd-8350-2bb7d19e6e7a/dd51c51a-fa64-4ebf-8f16-6468af1aee8c"
-					(reference "C4")
+					(reference "C8")
 					(unit 1)
 				)
@@
 		(on_board yes)
 		(dnp no)
-		(property "Reference" "#PWR08"
+		(property "Reference" "#PWR019"
 			(at 256.54 82.55 0)
 			(effects
@@
 			(project "PACS_1.0"
 				(path "/6996cbc8-fffb-40fd-8350-2bb7d19e6e7a/dd51c51a-fa64-4ebf-8f16-6468af1aee8c"
-					(reference "#PWR08")
+					(reference "#PWR019")
 					(unit 1)
 				)
@@
 		(dnp no)
 		(fields_autoplaced yes)
-		(property "Reference" "#PWR027"
+		(property "Reference" "#PWR012"
 			(at 41.91 119.38 0)
 			(effects
@@
 			(project "PACS_1.0"
 				(path "/6996cbc8-fffb-40fd-8350-2bb7d19e6e7a/dd51c51a-fa64-4ebf-8f16-6468af1aee8c"
-					(reference "#PWR027")
+					(reference "#PWR012")
 					(unit 1)
 				)
@@
 		(dnp no)
 		(fields_autoplaced yes)
-		(property "Reference" "C6"
+		(property "Reference" "C10"
 			(at 266.7 64.7699 0)
 			(effects
@@
 			(project "PACS_1.0"
 				(path "/6996cbc8-fffb-40fd-8350-2bb7d19e6e7a/dd51c51a-fa64-4ebf-8f16-6468af1aee8c"
-					(reference "C6")
+					(reference "C10")
 					(unit 1)
 				)
@@
 		(dnp no)
 		(fields_autoplaced yes)
-		(property "Reference" "Q2"
+		(property "Reference" "Q1"
 			(at 184.15 125.7299 0)
 			(effects
@@
 			(project ""
 				(path "/6996cbc8-fffb-40fd-8350-2bb7d19e6e7a/dd51c51a-fa64-4ebf-8f16-6468af1aee8c"
-					(reference "Q2")
+					(reference "Q1")
 					(unit 1)
 				)
@@
 		(dnp no)
 		(fields_autoplaced yes)
-		(property "Reference" "#PWR037"
+		(property "Reference" "#PWR013"
 			(at 166.37 154.94 0)
 			(effects
@@
 			(project "PACS_1.0"
 				(path "/6996cbc8-fffb-40fd-8350-2bb7d19e6e7a/dd51c51a-fa64-4ebf-8f16-6468af1aee8c"
-					(reference "#PWR037")
+					(reference "#PWR013")
 					(unit 1)
 				)
@@
 		(dnp no)
 		(fields_autoplaced yes)
-		(property "Reference" "U7"
+		(property "Reference" "U3"
 			(at 209.55 115.1902 0)
 			(effects
@@
 			(project ""
 				(path "/6996cbc8-fffb-40fd-8350-2bb7d19e6e7a/dd51c51a-fa64-4ebf-8f16-6468af1aee8c"
-					(reference "U7")
+					(reference "U3")
 					(unit 1)
 				)
@@
 		(dnp no)
 		(fields_autoplaced yes)
-		(property "Reference" "R17"
+		(property "Reference" "R7"
 			(at 168.91 133.3499 0)
 			(effects
@@
 			(project "PACS_1.0"
 				(path "/6996cbc8-fffb-40fd-8350-2bb7d19e6e7a/dd51c51a-fa64-4ebf-8f16-6468af1aee8c"
-					(reference "R17")
+					(reference "R7")
 					(unit 1)
 				)
@@
 		(dnp no)
 		(fields_autoplaced yes)
-		(property "Reference" "R16"
+		(property "Reference" "R12"
 			(at 208.28 143.5099 0)
 			(effects
@@
 			(project "PACS_1.0"
 				(path "/6996cbc8-fffb-40fd-8350-2bb7d19e6e7a/dd51c51a-fa64-4ebf-8f16-6468af1aee8c"
-					(reference "R16")
+					(reference "R12")
 					(unit 1)
 				)
@@
 		(dnp no)
 		(fields_autoplaced yes)
-		(property "Reference" "R1"
+		(property "Reference" "R10"
 			(at 186.69 69.8499 0)
 			(effects
@@
 			(project ""
 				(path "/6996cbc8-fffb-40fd-8350-2bb7d19e6e7a/dd51c51a-fa64-4ebf-8f16-6468af1aee8c"
-					(reference "R1")
+					(reference "R10")
 					(unit 1)
 				)
@@
 		(on_board yes)
 		(dnp no)
-		(property "Reference" "C5"
+		(property "Reference" "C9"
 			(at 254 64.7699 0)
 			(effects
@@
 			(project ""
 				(path "/6996cbc8-fffb-40fd-8350-2bb7d19e6e7a/dd51c51a-fa64-4ebf-8f16-6468af1aee8c"
-					(reference "C5")
+					(reference "C9")
 					(unit 1)
 				)
@@
 		(dnp no)
 		(fields_autoplaced yes)
-		(property "Reference" "#PWR09"
+		(property "Reference" "#PWR014"
 			(at 168.91 20.32 0)
 			(effects
@@
 			(project "PACS_1.0"
 				(path "/6996cbc8-fffb-40fd-8350-2bb7d19e6e7a/dd51c51a-fa64-4ebf-8f16-6468af1aee8c"
-					(reference "#PWR09")
+					(reference "#PWR014")
 					(unit 1)
 				)
@@
 		(dnp no)
 		(fields_autoplaced yes)
-		(property "Reference" "U2"
+		(property "Reference" "U4"
 			(at 210.82 40.64 0)
 			(effects
@@
 			(project ""
 				(path "/6996cbc8-fffb-40fd-8350-2bb7d19e6e7a/dd51c51a-fa64-4ebf-8f16-6468af1aee8c"
-					(reference "U2")
+					(reference "U4")
 					(unit 1)
 				)
@@
 		(on_board yes)
 		(dnp no)
-		(property "Reference" "R2"
+		(property "Reference" "R8"
 			(at 176.784 70.104 0)
 			(effects
@@
 			(project "PACS_1.0"
 				(path "/6996cbc8-fffb-40fd-8350-2bb7d19e6e7a/dd51c51a-fa64-4ebf-8f16-6468af1aee8c"
-					(reference "R2")
+					(reference "R8")
 					(unit 1)
 				)
@@
 		(dnp no)
 		(fields_autoplaced yes)
-		(property "Reference" "#PWR036"
+		(property "Reference" "#PWR017"
 			(at 205.74 157.48 0)
 			(effects
@@
 			(project "PACS_1.0"
 				(path "/6996cbc8-fffb-40fd-8350-2bb7d19e6e7a/dd51c51a-fa64-4ebf-8f16-6468af1aee8c"
-					(reference "#PWR036")
+					(reference "#PWR017")
 					(unit 1)
 				)
@@
 		(dnp no)
 		(fields_autoplaced yes)
-		(property "Reference" "#PWR012"
+		(property "Reference" "#PWR011"
 			(at 33.02 73.66 0)
 			(effects
@@
 			(project "PACS_1.0"
 				(path "/6996cbc8-fffb-40fd-8350-2bb7d19e6e7a/dd51c51a-fa64-4ebf-8f16-6468af1aee8c"
-					(reference "#PWR012")
+					(reference "#PWR011")
 					(unit 1)
 				)
@@
 		(dnp no)
 		(fields_autoplaced yes)
-		(property "Reference" "#PWR07"
+		(property "Reference" "#PWR016"
 			(at 184.15 83.82 0)
 			(effects
@@
 			(project "PACS_1.0"
 				(path "/6996cbc8-fffb-40fd-8350-2bb7d19e6e7a/dd51c51a-fa64-4ebf-8f16-6468af1aee8c"
-					(reference "#PWR07")
+					(reference "#PWR016")
 					(unit 1)
 				)
@@
 		(dnp no)
 		(fields_autoplaced yes)
-		(property "Reference" "C7"
+		(property "Reference" "C5"
 			(at 160.02 39.3701 0)
 			(effects
@@
 			(project "PACS_1.0"
 				(path "/6996cbc8-fffb-40fd-8350-2bb7d19e6e7a/dd51c51a-fa64-4ebf-8f16-6468af1aee8c"
-					(reference "C7")
+					(reference "C5")
 					(unit 1)
 				)
@@
 		(dnp no)
 		(fields_autoplaced yes)
-		(property "Reference" "R15"
+		(property "Reference" "R11"
 			(at 208.28 128.2699 0)
 			(effects
@@
 			(project "PACS_1.0"
 				(path "/6996cbc8-fffb-40fd-8350-2bb7d19e6e7a/dd51c51a-fa64-4ebf-8f16-6468af1aee8c"
-					(reference "R15")
+					(reference "R11")
 					(unit 1)
 				)
@@
 		(dnp no)
 		(fields_autoplaced yes)
-		(property "Reference" "R10"
+		(property "Reference" "R9"
 			(at 184.15 106.6799 0)
 			(effects
@@
 			(project ""
 				(path "/6996cbc8-fffb-40fd-8350-2bb7d19e6e7a/dd51c51a-fa64-4ebf-8f16-6468af1aee8c"
-					(reference "R10")
+					(reference "R9")
 					(unit 1)
 				)
@@
 		(dnp no)
 		(fields_autoplaced yes)
-		(property "Reference" "C9"
+		(property "Reference" "C7"
 			(at 185.42 39.3701 0)
 			(effects
@@
 			(project "PACS_1.0"
 				(path "/6996cbc8-fffb-40fd-8350-2bb7d19e6e7a/dd51c51a-fa64-4ebf-8f16-6468af1aee8c"
-					(reference "C9")
+					(reference "C7")
 					(unit 1)
 				)
@@
 		(dnp no)
 		(fields_autoplaced yes)
-		(property "Reference" "U8"
+		(property "Reference" "U2"
 			(at 57.15 93.98 0)
 			(effects
@@
 			(project ""
 				(path "/6996cbc8-fffb-40fd-8350-2bb7d19e6e7a/dd51c51a-fa64-4ebf-8f16-6468af1aee8c"
-					(reference "U8")
-					(unit 1)
-				)
+					(reference "U2")
+					(unit 1)
+				)

Commit message: Changed 5.5k resistor to 5.49k
Parts:
- R11: value 5.5k -> 5.49k
Changed lines of the file:
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@@
 			)
 		)
-		(property "Value" "5.5k"
+		(property "Value" "5.49k"
 			(at 208.28 130.8099 0)
 			(effects

Commit message: Added Boxes and fixed PDF
Other:
- note added: "Buck Converter"
- note added: "Switchable Voltage Divider"
- moved on the sheet: C10, C5, C6, C7, C8, C9, L1, R10, R6, R8, U4

Commit message: Updated footprints for caps and resistors
Parts:
- C10, C9: footprint (none) -> Capacitor_SMD:C_0603_1608Metric
- C5, C6: footprint (none) -> Capacitor_SMD:C_0805_2012Metric
- C7, C8: footprint (none) -> Capacitor_SMD:C_0402_1005Metric
- R10, R4, R5, R6, R7, R8, R9: footprint (none) -> Resistor_SMD:R_0402_1005Metric
- R11, R12: footprint (none) -> Resistor_SMD:R_0603_1608Metric
Changed lines of the file:
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@@
 			)
 		)
-		(property "Footprint" ""
+		(property "Footprint" "Resistor_SMD:R_0402_1005Metric"
 			(at 162.56 55.118 90)
 			(effects
@@
 			)
 		)
-		(property "Footprint" ""
+		(property "Footprint" "Capacitor_SMD:C_0805_2012Metric"
 			(at 166.0652 34.29 0)
 			(effects
@@
 			)
 		)
-		(property "Footprint" ""
+		(property "Footprint" "Resistor_SMD:R_0402_1005Metric"
 			(at 156.21 128.778 90)
 			(effects
@@
 			)
 		)
-		(property "Footprint" ""
+		(property "Footprint" "Resistor_SMD:R_0402_1005Metric"
 			(at 97.028 101.6 90)
 			(effects
@@
 			)
 		)
-		(property "Footprint" ""
+		(property "Footprint" "Capacitor_SMD:C_0402_1005Metric"
 			(at 212.09 76.5048 0)
 			(effects
@@
 			)
 		)
-		(property "Footprint" ""
+		(property "Footprint" "Capacitor_SMD:C_0603_1608Metric"
 			(at 260.0452 69.85 0)
 			(effects
@@
 			)
 		)
-		(property "Footprint" ""
+		(property "Footprint" "Resistor_SMD:R_0402_1005Metric"
 			(at 164.592 134.62 90)
 			(effects
@@
 			)
 		)
-		(property "Footprint" ""
+		(property "Footprint" "Resistor_SMD:R_0603_1608Metric"
 			(at 203.962 144.78 90)
 			(effects
@@
 			)
 		)
-		(property "Footprint" ""
+		(property "Footprint" "Resistor_SMD:R_0402_1005Metric"
 			(at 178.562 71.12 90)
 			(effects
@@
 			)
 		)
-		(property "Footprint" ""
+		(property "Footprint" "Capacitor_SMD:C_0603_1608Metric"
 			(at 247.3452 69.85 0)
 			(effects
@@
 			)
 		)
-		(property "Footprint" ""
+		(property "Footprint" "Resistor_SMD:R_0402_1005Metric"
 			(at 167.132 71.12 90)
 			(effects
@@
 			)
 		)
-		(property "Footprint" ""
+		(property "Footprint" "Capacitor_SMD:C_0805_2012Metric"
 			(at 153.3652 34.29 0)
 			(effects
@@
 			)
 		)
-		(property "Footprint" ""
+		(property "Footprint" "Resistor_SMD:R_0603_1608Metric"
 			(at 203.962 129.54 90)
 			(effects
@@
 			)
 		)
-		(property "Footprint" ""
+		(property "Footprint" "Resistor_SMD:R_0402_1005Metric"
 			(at 179.832 107.95 90)
 			(effects
@@
 			)
 		)
-		(property "Footprint" ""
+		(property "Footprint" "Capacitor_SMD:C_0402_1005Metric"
 			(at 178.7652 34.29 0)
 			(effects

Commit message: added more footprints
Parts:
- U3: footprint BSS84PH6327XTSA2:SOT-23-3 -> Package_TO_SOT_SMD:SOT-23-5_HandSoldering
Changed lines of the file:
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@@
 			)
 		)
-		(property "Footprint" "BSS84PH6327XTSA2:SOT-23-3"
+		(property "Footprint" "Package_TO_SOT_SMD:SOT-23-5_HandSoldering"
 			(at 203.2 116.84 0)
 			(effects

Commit message: Started the PCB design
added several footprints, need to find footprint for Xbee, need to add traces for GND and power
Parts:
- BT1: footprint (none) -> Connector_JST:JST_EH_B2B-EH-A_1x02_P2.50mm_Vertical
- F1: footprint (none) -> Fuse:Fuse_1812_4532Metric
- L1: footprint (none) -> Inductor_SMD:L_Abracon_ASPI-0630LR
Changed lines of the file:
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@@
 			)
 		)
-		(property "Footprint" ""
+		(property "Footprint" "Connector_JST:JST_EH_B2B-EH-A_1x02_P2.50mm_Vertical"
 			(at 33.02 55.626 90)
 			(effects
@@
 			)
 		)
-		(property "Footprint" ""
+		(property "Footprint" "Fuse:Fuse_1812_4532Metric"
 			(at 67.31 49.53 0)
 			(effects
@@
 			)
 		)
-		(property "Footprint" ""
+		(property "Footprint" "Inductor_SMD:L_Abracon_ASPI-0630LR"
 			(at 238.76 58.42 0)
 			(effects
