File: PACS_1.0/PACS_1.0_power.kicad_sch (KiCad schematic)
At the start: 22 parts, among them Q1 PN2222A, U2 S-80855CNMC-B9GT2U, U3 BSS84PH6327XTSA2, U4 TPS562201DDCR

Commit message: FINISHED PCB DESIGN
must double check that the dimensions for XBee footprint are correct
Parts:
- U3: footprint Package_TO_SOT_SMD:SOT-23-5_HandSoldering -> Package_TO_SOT_SMD:TSOT-23
Changed lines of the file:
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@@
 			)
 		)
-		(property "Footprint" "Package_TO_SOT_SMD:SOT-23-5_HandSoldering"
+		(property "Footprint" "Package_TO_SOT_SMD:TSOT-23"
 			(at 203.2 116.84 0)
 			(effects
